File: PB450-riser.kicad_pcb (KiCad board)
At the start: 4 copper layers, 160 x 81.3 mm, 29 parts, among them J1 J1, J2 J1, J3 J1, P1 ISA Bus over PCI

Commit message: Fixed small bug in PCI footprint
Parts:
- added P2: PCI 32bit footprint (partial), Connector_PCBEdge:BUS_PCI, F.Cu at (40.3, 5.17)
- moved C12 0.19 mm to (129.5, 89.6)
Connections:
- net Net-(J1-AEN) renamed /AEN
- net Net-(J1-IO_CH_RDY) renamed /IO_CH_RDY
- net Net-(J1-SBHE) renamed /SBHE
- net Net-(J1-~{IO_CH_CK}) renamed //IO_CH_CLK
- net Net-(J1-~{MEMR}) renamed //MEMR
- net Net-(J1-~{MEMW}) renamed //MEMW
- C11 pad 1: +5V -> GND
- C11 pad 2: GND -> +12V
- C12 pad 1: +5V -> +12V
- P1 pad B20: Net-(J1-~{REFRESH}) -> Net-(J1-SYSCLK)
- P1 pad B21: Net-(J1-SYSCLK) -> Net-(J1-IRQ7)
- P1 pad B22: Net-(J1-IRQ7) -> Net-(J1-IRQ6)
- P1 pad B23: Net-(J1-IRQ6) -> Net-(J1-IRQ5)
- P1 pad B24: Net-(J1-IRQ5) -> Net-(J1-IRQ4)
- P1 pad B25: Net-(J1-IRQ4) -> Net-(J1-IRQ3)
- P1 pad B26: Net-(J1-IRQ3) -> Net-(J1-~{DACK2})
- P1 pad B27: Net-(J1-~{DACK2}) -> Net-(J1-TC)
- P1 pad B28: Net-(J1-TC) -> Net-(J1-BALE)
Routing:
- net Net-(J1-BALE): track 41.8 -> 82.7 mm, vias 0 -> 5
- net +12V: track 90.7 -> 124.0 mm
- net +5V: track 779.9 -> 756.9 mm, vias 12 -> 11
- net Net-(J1-IRQ4): track 81.4 -> 82.4 mm
- net Net-(J1-IRQ7): track 104.0 -> 104.9 mm
- net Net-(J1-IRQ6): track 116.2 -> 116.7 mm
- net Net-(J1-~{DACK2}): track 123.4 -> 122.8 mm
- net Net-(J1-IRQ5): track 126.7 -> 127.3 mm
